File: gravity/gravity.kicad_sch (KiCad schematic)
At the start: 78 parts, among them Q1 IRF820, Q2 IRF820, SW1 SW_SPST, U1 6N2P, U2 6N2P, U3 6N2P

Commit message: tube ressurection
Parts:
- C5: value 1n -> 22n
Changed lines of the file:
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@@
 			)
 		)
-		(property "Value" "1n"
+		(property "Value" "22n"
 			(at 162.56 46.99 90)
 			(effects

Commit message: gravity with supply
Parts:
- added C22, C23: 10n, symbol Device:C
- added C24: 220n, symbol Device:C
- added C25, C26: 22n, symbol Device:C
- added J3: ~, symbol Connector_Audio:AudioJack3_Switch
- added R41: 10k, symbol Device:R
- added RV5: 1M, symbol Device:R_Potentiometer
- C21: value 100n -> 220n
- C5: value 22n -> 220n
Connections:
- net TO_CC_SW is gone; now on an unnamed net: C9.2
- net GND: now also J3.S
- net at D1.2 (A), D2.1 (K), SW1.1 (A)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: now also RV5.1; no longer SW2.6 (C)
- net at R19.2, R20.1: now also C24.2; no longer SW4.5 (B)
- net at R27.1: now also C26.2; no longer SW5.5 (B)
- net at R5.2, R6.2: now also C22.2; no longer SW2.2 (B)
- net at SW5.2 (B): now also C25.1; no longer R23.1
- net at SW4.2 (B): now also C23.1; no longer R11.1
- net 2: now reaches C18.2
- net FROM_GS1: no longer names the net of SW5.1 (A), SW5.6 (C)
- new net: R41.1, RV5.2, SW2.6 (C)
- new net: C22.1, SW2.2 (B)
- new net: C26.1, SW5.5 (B)
- new net: C25.2, R23.1
- new net: R41.2, RV5.3
- new net: C23.2, R11.1
- new net 1: C24.1, SW4.5 (B)
- new net OUT: J3.T
Other:
- added sheet PSU (untitled.kicad_sch)
- added sheet TONE_BLOCK (tone.kicad_sch)
- moved on the sheet: C10, C11, C12, C14, C15, C16, C17, C19, C20, C21, C4, C5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

Commit message: pre mark II soldering
Other:
- moved on the sheet: C18
Changed lines of the file:
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@@
 	)
 	(junction
+		(at 317.5 156.21)
+		(diameter 0)
+		(color 0 0 0 0)
+	)
+	(junction
 		(at 313.69 73.66)
 		(diameter 0)
@@
 	)
 	(junction
-		(at 328.93 156.21)
-		(diameter 0)
-		(color 0 0 0 0)
-	)
-	(junction
 		(at 290.83 54.61)
 		(diameter 0)
@@
 	)
 	(junction
-		(at 317.5 156.21)
-		(diameter 0)
-		(color 0 0 0 0)
-	)
-	(junction
 		(at 172.72 52.07)
 		(diameter 0)
@@
 	(wire
 		(pts
-			(xy 317.5 156.21) (xy 321.31 156.21)
-		)
-		(stroke
-			(width 0)
-			(type default)
-		)
-	)
-	(wire
-		(pts
 			(xy 290.83 46.99) (xy 290.83 54.61)
 		)
@@
 	(wire
 		(pts
-			(xy 317.5 148.59) (xy 317.5 156.21)
-		)
-		(stroke
-			(width 0)
-			(type default)
-		)
-	)
-	(wire
-		(pts
 			(xy 285.75 170.18) (xy 285.75 172.72)
 		)
@@
 	(wire
 		(pts
-			(xy 317.5 156.21) (xy 317.5 160.02)
+			(xy 317.5 148.59) (xy 317.5 156.21)
 		)
 		(stroke
@@
 	(wire
 		(pts
-			(xy 328.93 156.21) (xy 335.28 156.21)
-		)
-		(stroke
-			(width 0)
-			(type default)
-		)
-	)
-	(wire
-		(pts
 			(xy 170.18 73.66) (xy 170.18 76.2)
 		)
@@
 	(wire
 		(pts
+			(xy 317.5 156.21) (xy 320.04 156.21)
+		)
+		(stroke
+			(width 0)
+			(type default)
+		)
+	)
+	(wire
+		(pts
 			(xy 93.98 151.13) (xy 93.98 153.67)
 		)
@@
 	(wire
 		(pts
+			(xy 327.66 156.21) (xy 335.28 156.21)
+		)
+		(stroke
+			(width 0)
+			(type default)
+		)
+	)
+	(wire
+		(pts
 			(xy 326.39 72.39) (xy 326.39 87.63)
 		)
@@
 	(wire
 		(pts
-			(xy 322.58 156.21) (xy 328.93 156.21)
-		)
-		(stroke
-			(width 0)
-			(type default)
-		)
-	)
-	(wire
-		(pts
 			(xy 153.67 63.5) (xy 153.67 68.58)
 		)
@@
 	(wire
 		(pts
+			(xy 317.5 156.21) (xy 317.5 160.02)
+		)
+		(stroke
+			(width 0)
+			(type default)
+		)
+	)
+	(wire
+		(pts
 			(xy 77.47 71.12) (xy 77.47 73.66)
 		)
@@
 	(symbol
 		(lib_id "Device:C")
-		(at 325.12 156.21 90)
+		(at 323.85 156.21 90)
 		(unit 1)
 		(exclude_from_sim no)
@@
 		(on_board yes)
 		(dnp no)
-		(fields_autoplaced yes)
 		(property "Reference" "C18"
-			(at 325.12 148.59 90)
+			(at 323.85 148.59 90)
 			(effects
 				(font
@@
 		)
 		(property "Value" "µ1"
-			(at 325.12 151.13 90)
+			(at 323.85 151.13 90)
 			(effects
 				(font
@@
 		)
 		(property "Footprint" ""
-			(at 328.93 155.2448 0)
+			(at 327.66 155.2448 0)
 			(effects
 				(font
@@
 		)
 		(property "Datasheet" "~"
-			(at 325.12 156.21 0)
+			(at 323.85 156.21 0)
 			(effects
 				(font
@@
 		)
 		(property "Description" ""
-			(at 325.12 156.21 0)
+			(at 323.85 156.21 0)
 			(effects
 				(font

Commit message: pre actual tonestack
Parts:
- removed D3, D4: 1N914, Diode_THT:D_DO-35_SOD27_P7.62mm_Horizontal, symbol Diode:1N914
- removed SW3: ~, symbol Switch:SW_SPST
- added C35: 1n, symbol Device:C
- R25: value 39K -> 20K
Connections:
- net GND: now also C35.1
- net at R10.2, R6.1, U1.2 (G): now also C35.2
