File: gravity/tone.kicad_sch (KiCad schematic)
At the start: 8 parts

Commit message: pre mark II soldering
Parts:
- renumbered RB to RB1, RM to RM1, RT to RT1, VOL to VOL1
Changed lines of the file:
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@@
 		(dnp no)
 		(fields_autoplaced yes)
-		(property "Reference" "VOL"
+		(property "Reference" "VOL1"
 			(at 90.17 60.9599 0)
 			(effects
@@
 			(project "gravity"
 				(path "/aa56c72d-d58e-465d-9854-f9d2b610c8e6/c5d4d34a-f0e5-4d7f-9edb-fbac8bc75ba1"
-					(reference "VOL")
+					(reference "VOL1")
 					(unit 1)
 				)
@@
 		(dnp no)
 		(fields_autoplaced yes)
-		(property "Reference" "RT"
+		(property "Reference" "RT1"
 			(at 62.23 39.3699 0)
 			(effects
@@
 			(project ""
 				(path "/aa56c72d-d58e-465d-9854-f9d2b610c8e6/c5d4d34a-f0e5-4d7f-9edb-fbac8bc75ba1"
-					(reference "RT")
+					(reference "RT1")
 					(unit 1)
 				)
@@
 		(dnp no)
 		(fields_autoplaced yes)
-		(property "Reference" "RB"
+		(property "Reference" "RB1"
 			(at 62.23 62.2299 0)
 			(effects
@@
 			(project ""
 				(path "/aa56c72d-d58e-465d-9854-f9d2b610c8e6/c5d4d34a-f0e5-4d7f-9edb-fbac8bc75ba1"
-					(reference "RB")
+					(reference "RB1")
 					(unit 1)
 				)
@@
 		(on_board yes)
 		(dnp no)
-		(property "Reference" "RM"
+		(property "Reference" "RM1"
 			(at 67.31 77.4699 0)
 			(effects
@@
 			(project ""
 				(path "/aa56c72d-d58e-465d-9854-f9d2b610c8e6/c5d4d34a-f0e5-4d7f-9edb-fbac8bc75ba1"
-					(reference "RM")
-					(unit 1)
-				)
+					(reference "RM1")
+					(unit 1)
+				)

Commit message: pre actual tonestack
Parts:
- R44: value 47k -> 100k
- RB1: value 250k -> B250k
- RM1: value 25k -> B25k
- RT1: value 250k -> A250k
Changed lines of the file:
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@@
 			)
 		)
-		(property "Value" "250k"
+		(property "Value" "A250k"
 			(at 62.23 41.9099 0)
 			(effects
@@
 			)
 		)
-		(property "Value" "47k"
+		(property "Value" "100k"
 			(at 43.18 45.7199 0)
 			(effects
@@
 			)
 		)
-		(property "Value" "250k"
+		(property "Value" "B250k"
 			(at 62.23 64.7699 0)
 			(effects
@@
 			)
 		)
-		(property "Value" "25k"
+		(property "Value" "B25k"
 			(at 67.31 80.0099 0)
 			(effects
