File: gravity/untitled.kicad_sch (KiCad schematic)
At the start: 26 parts, among them J2 IEC_60320_C14_Receptacle, T2 Transformer_1P_3S, U1 6N2P, U2 6N2P, U3 6N2P, U5 LM7805_TO220

Commit message: pre mark II soldering
Parts:
- C27: footprint (none) -> Capacitor_THT:CP_Radial_D24.0mm_P10.00mm_SnapIn
- C28: value C_Polarized -> 1000u; footprint (none) -> Capacitor_THT:CP_Radial_D16.0mm_P7.50mm
- C29: value C_Polarized -> 4700u; footprint (none) -> Capacitor_THT:CP_Radial_D16.0mm_P7.50mm
- C30, C31: footprint (none) -> Capacitor_THT:CP_Radial_D22.0mm_P10.00mm_SnapIn
- D11, D12, D13, D14, D15, D16, D17, D18: footprint (none) -> Diode_THT:D_DO-41_SOD81_P10.16mm_Horizontal
- R39, R40: footprint (none) -> Resistor_THT:R_Axial_DIN0614_L14.3mm_D5.7mm_P20.32mm_Horizontal
- R42, R43: footprint (none) -> Resistor_THT:R_Axial_DIN0309_L9.0mm_D3.2mm_P12.70mm_Horizontal
Changed lines of the file:
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@@
 			)
 		)
-		(property "Footprint" ""
+		(property "Footprint" "Diode_THT:D_DO-41_SOD81_P10.16mm_Horizontal"
 			(at 196.85 41.91 0)
 			(effects
@@
 			)
 		)
-		(property "Footprint" ""
+		(property "Footprint" "Diode_THT:D_DO-41_SOD81_P10.16mm_Horizontal"
 			(at 82.55 46.99 0)
 			(effects
@@
 			)
 		)
-		(property "Footprint" ""
+		(property "Footprint" "Resistor_THT:R_Axial_DIN0309_L9.0mm_D3.2mm_P12.70mm_Horizontal"
 			(at 100.838 87.63 90)
 			(effects
@@
 			)
 		)
-		(property "Footprint" ""
+		(property "Footprint" "Diode_THT:D_DO-41_SOD81_P10.16mm_Horizontal"
 			(at 191.77 46.99 0)
 			(effects
@@
 			)
 		)
-		(property "Footprint" ""
+		(property "Footprint" "Diode_THT:D_DO-41_SOD81_P10.16mm_Horizontal"
 			(at 191.77 41.91 0)
 			(effects
@@
 			)
 		)
-		(property "Footprint" ""
+		(property "Footprint" "Capacitor_THT:CP_Radial_D24.0mm_P10.00mm_SnapIn"
 			(at 98.7552 54.61 0)
 			(effects
@@
 			)
 		)
-		(property "Footprint" ""
+		(property "Footprint" "Diode_THT:D_DO-41_SOD81_P10.16mm_Horizontal"
 			(at 196.85 46.99 0)
 			(effects
@@
 			)
 		)
-		(property "Footprint" ""
+		(property "Footprint" "Resistor_THT:R_Axial_DIN0309_L9.0mm_D3.2mm_P12.70mm_Horizontal"
 			(at 100.838 78.74 90)
 			(effects
@@
 			)
 		)
-		(property "Footprint" ""
+		(property "Footprint" "Diode_THT:D_DO-41_SOD81_P10.16mm_Horizontal"
 			(at 82.55 41.91 0)
 			(effects
@@
 			)
 		)
-		(property "Footprint" ""
+		(property "Footprint" "Diode_THT:D_DO-41_SOD81_P10.16mm_Horizontal"
 			(at 77.47 41.91 0)
 			(effects
@@
 			)
 		)
-		(property "Value" "C_Polarized"
+		(property "Value" "4700u"
 			(at 248.92 58.8009 0)
 			(effects
@@
 			)
 		)
-		(property "Footprint" ""
+		(property "Footprint" "Capacitor_THT:CP_Radial_D16.0mm_P7.50mm"
 			(at 246.0752 62.23 0)
 			(effects
@@
 			)
 		)
-		(property "Footprint" ""
+		(property "Footprint" "Resistor_THT:R_Axial_DIN0614_L14.3mm_D5.7mm_P20.32mm_Horizontal"
 			(at 134.62 46.228 90)
 			(effects
@@
 			)
 		)
-		(property "Footprint" ""
+		(property "Footprint" "Diode_THT:D_DO-41_SOD81_P10.16mm_Horizontal"
 			(at 77.47 46.99 0)
 			(effects
@@
 			)
 		)
-		(property "Footprint" ""
+		(property "Footprint" "Resistor_THT:R_Axial_DIN0614_L14.3mm_D5.7mm_P20.32mm_Horizontal"
 			(at 109.22 46.228 90)
 			(effects
@@
 			)
 		)
-		(property "Footprint" ""
+		(property "Footprint" "Capacitor_THT:CP_Radial_D22.0mm_P10.00mm_SnapIn"
 			(at 147.0152 54.61 0)
 			(effects
@@
 			)
 		)
-		(property "Footprint" ""
+		(property "Footprint" "Capacitor_THT:CP_Radial_D22.0mm_P10.00mm_SnapIn"
 			(at 124.1552 54.61 0)
 			(effects
@@
 			)
 		)
-		(property "Value" "C_Polarized"
+		(property "Value" "1000u"
 			(at 208.28 58.8009 0)
 			(effects
@@
 			)
 		)
-		(property "Footprint" ""
+		(property "Footprint" "Capacitor_THT:CP_Radial_D16.0mm_P7.50mm"
 			(at 205.4352 62.23 0)
 			(effects

Commit message: pre actual tonestack
Parts:
- added C36: 100u, Capacitor_THT:CP_Radial_D24.0mm_P10.00mm_SnapIn, symbol Device:C_Polarized
- added R45: 1k, Resistor_THT:R_Axial_DIN0614_L14.3mm_D5.7mm_P20.32mm_Horizontal, symbol Device:R
- added R46: 150, Resistor_THT:R_Axial_DIN0614_L14.3mm_D5.7mm_P20.32mm_Horizontal, symbol Device:R
- C30, C31: value 47u -> 100u
- F1: value T100ma -> T500ma
Connections:
- net +A: now also R45.1; no longer C27.1, D11.1 (K), D12.1 (K)
- net GND: now also C36.2
- new net: C36.1, D11.1 (K), D12.1 (K), R46.2
- new net: C27.1, R45.2, R46.1
Other:
- moved on the sheet: C30, C31, R39, R40
