File: LockUp/LockUp.kicad_sch (KiCad schematic)
At the start: 4 parts, among them J1 Conn_01x05_Socket, J2 Conn_01x02_Socket, U1 ESP32-C6-WROOM-1

Commit message: pwr
Parts:
- removed J1: Conn_01x05_Socket, symbol Connector:Conn_01x05_Socket
- added 10K1: NR14, Resistor_SMD:R_0805_2012Metric_Pad1.20x1.40mm_HandSolder, symbol Device:R
- added 300R1: NR18, Resistor_SMD:R_0805_2012Metric_Pad1.20x1.40mm_HandSolder, symbol Device:R
- added 300R2: NR17, Resistor_SMD:R_0805_2012Metric_Pad1.20x1.40mm_HandSolder, symbol Device:R
- added 5K1: NR16, Resistor_SMD:R_0805_2012Metric_Pad1.20x1.40mm_HandSolder, symbol Device:R
- added 820R1: NR15, Resistor_SMD:R_0805_2012Metric_Pad1.20x1.40mm_HandSolder, symbol Device:R
- added J4: Key_Sw, Connector_Molex:Molex_PicoBlade_53398-0271_1x02-1MP_P1.25mm_Vertical, symbol Connector:Conn_01x02_Socket
- added J5: DND_sw, Connector_Molex:Molex_PicoBlade_53398-0271_1x02-1MP_P1.25mm_Vertical, symbol Connector:Conn_01x02_Socket
- added J7: Servo, symbol Connector:Conn_01x03_Socket
- added LS1: Speaker, Buzzer_Beeper:Buzzer_Mallory_AST1240MLQ, symbol Device:Speaker
- added NC16, NC17, NC18, NC19: 15pF, Capacitor_SMD:C_0805_2012Metric_Pad1.18x1.45mm_HandSolder, symbol Device:C
- added NC20, NC21: 180pF, Capacitor_SMD:C_0805_2012Metric_Pad1.18x1.45mm_HandSolder, symbol Device:C
- added NC22, NC23: 10pF, Capacitor_SMD:C_0805_2012Metric_Pad1.18x1.45mm_HandSolder, symbol Device:C
- added NC24, NC25: 47pF, Capacitor_SMD:C_0805_2012Metric_Pad1.18x1.45mm_HandSolder, symbol Device:C
- added NC26, NC27, NC5, NC6: 100nF, Capacitor_SMD:C_0805_2012Metric_Pad1.18x1.45mm_HandSolder, symbol Device:C
- added NL4, NL5: 22uH, Inductor_SMD:L_0805_2012Metric_Pad1.15x1.40mm_HandSolder, symbol Device:L
- added NT1: CLK, TestPoint:TestPoint_Pad_1.0x1.0mm, symbol Connector:TestPoint
- added NT2: MO, TestPoint:TestPoint_Pad_1.0x1.0mm, symbol Connector:TestPoint
- added NT3: MI, TestPoint:TestPoint_Pad_1.0x1.0mm, symbol Connector:TestPoint
- added NT4: DA, TestPoint:TestPoint_Pad_1.0x1.0mm, symbol Connector:TestPoint
- added NT5: 3V3, TestPoint:TestPoint_Pad_1.0x1.0mm, symbol Connector:TestPoint
- added NT6: GND, TestPoint:TestPoint_Pad_1.0x1.0mm, symbol Connector:TestPoint
- added NY1: 27M12, Crystal:Crystal_SMD_3225-4Pin_3.2x2.5mm_HandSoldering, symbol Device:Crystal_GND24
- added R1, R2: R, symbol Device:R
- added U3: MFRC522/RC522, Package_QFP:RC522 RFID NFC QFN50P500X500X100-33N, symbol RFID:MFRC522{brace}slash}RC522
- added U4: L9110S, Package_SO:SOP-8_3.9x4.9mm_P1.27mm, symbol OrnexParts:L9110S
- J2: value Conn_01x02_Socket -> Motor; footprint (none) -> Connector_Molex:Molex_PicoBlade_53398-0271_1x02-1MP_P1.25mm_Vertical
- U2: value ~ -> L9110S
Connections:
- net GND: now also J4.2 (Pin_2), J5.2 (Pin_2), J7.3 (Pin_3), NC16.2, NC17.2, NC20.2, NC21.1, NC22.2, NC23.1, NC24.2, NC25.1, NC26.2, NC27.2, NC5.2, NT6.1, NY1.2, NY1.4, U3.1 (I2C), U3.10 (TVSS), U3.14 (TVSS), U3.18 (AVSS), U3.4 (DVSS), U3.5 (PVSS), U4.5 (GND), U4.8 (GND)
- net VCC: now also 10K1.1, J7.2 (Pin_2), NC26.1, NC27.1, NT5.1, R1.1, R2.1, U3.12 (TVDD), U3.15 (AVDD), U3.2 (PVDD), U3.3 (DVDD), U3.32 (EA); no longer U2.2 (VCC), U2.3 (VCC)
- net MOSI: now reaches U1.7 (MTDO/GPIO7)
- net MOSI: now also NT2.1, U3.30 (D6/ADR_0/MOSI/MX)
- net CLK: now reaches U1.6 (MTCK/GPIO6/ADC1_CH6)
- net CLK: now also NT1.1, U3.29 (D5/ADR_1/SCK/DTRQ)
- net MISO: now reaches U1.5 (MTDI/GPIO5/ADC1_CH5)
- net MISO: now also NT3.1, U3.31 (D7/SCL/MISO/TX)
- net at U1.11 (GPIO10): now also J4.1 (Pin_1), R1.2
- net at U1.12 (GPIO11): now also J5.1 (Pin_1), R2.2
- net PIEZO: now reaches U1.16 (GPIO18)
- net PIEZO: now also U4.6 (IA)
- net at U1.23 (GPIO15): now also J7.1 (Pin_1)
- new net: 300R1.1, NC19.2, NC21.2, NC23.2
- new net: 300R2.1, NC18.2, NC20.1, NC22.1, NC6.2
- new net: 5K1.2, NC6.1
- new net: NC18.1, NC24.1, NL4.2
- new net: NC19.1, NC25.2, NL5.2
- new net: NC17.1, NY1.3, U3.22 (OSCOUT)
- new net: NC16.1, NY1.1, U3.21 (OSCIN)
- new net: 10K1.2, U3.6 (~{NRSTPD})
- new net: LS1.1, U4.1 (OA)
- new net: LS1.2, U4.4 (OB)
- new net +BATT: U2.2 (VCC), U2.3 (VCC), U4.2 (VCC), U4.3 (VCC)
- new net ANT_TX1: 300R2.2
- new net ANT_TX2: 300R1.2
- new net RX: 5K1.1, 820R1.2, U3.17 (RX)
- new net SDA: NT4.1, U3.24 (SDA/NSS/RX)
- new net TX1: NL4.1, U3.11 (TX1)
- new net TX2: NL5.1, U3.13 (TX2)
- new net VMID: 820R1.1, NC5.1, U3.16 (VMID)
- no-connect marks 0 -> 6
Other:
- added sheet PWR (conn.kicad_sch)
- note added: "LOW BATTERY CIRCUIT!"
- note added: "NOT PIEZO!"
- moved on the sheet: J2, U1, U2
