File: LockUp/LockUp.kicad_sch (KiCad schematic)
At the start: 64 parts, among them J1 JST_B8B, J2 USB_B_Mini, J7 Servo, Q4 Si2323, Q5 Si2323, Q6 AO3400A, SW1 RST, SW2 BOOT, SW3 NT_RST, T1 GND, T2 TX, T3 RX, T4 D+, T5 D-, T6 TX, T7 RES, U1 ESP32-C6-WROOM-1, U2 L9110S, U3 MFRC522{slash}RC522

Commit message: half done
Parts:
- T1, T4, T5: footprint TestPoint:TestPoint_Pad_1.0x1.0mm -> Ornex:TestPoint_THTPad_D0.6mm_Drill0.3mm
- T2, T3: footprint TestPoint:TestPoint_Pad_1.0x1.0mm -> TestPoint:TestPoint_Pad_D1.0mm
- T6: value TX -> VCC; footprint TestPoint:TestPoint_Pad_1.0x1.0mm -> Ornex:TestPoint_THTPad_D0.6mm_Drill0.3mm
Connections:
- net D+: no longer T4.1
- net D-: no longer T5.1
- net at J2.2 (D-), R19.2: now also T5.1
- net at J2.3 (D+), R18.2: now also T4.1
Other:
- moved on the sheet: R18, R19, T4, T5

Commit message: gate swaps...
Parts:
- removed J2: USB_B_Mini, Connector_USB:USB_Mini-B_Wuerth_65100516121_Horizontal, symbol Connector:USB_B_Mini
Connections:
- net USB_V+: now also T6.1
- net VCC: no longer T6.1
- net at U1.11 (GPIO10): now also U2.7 (IB); no longer U2.6 (IA)
- net at U1.12 (GPIO11): now also U2.6 (IA); no longer U2.7 (IB)
- net at C12.2, U2.4 (OB): now also J1.2 (Pin_2); no longer J1.1 (Pin_1)
- net at C12.1, U2.1 (OA): now also J1.1 (Pin_1); no longer J1.2 (Pin_2)
- no-connect marks 12 -> 10
Other:
- moved on the sheet: R18, R19, T1, T4, T5, T6

Commit message: frootloop day dream...
Parts:
- T7: footprint TestPoint:TestPoint_Pad_1.0x1.0mm -> TestPoint:TestPoint_Pad_D1.0mm
Connections:
- net at C12.1, U2.1 (OA): now also J1.2 (Pin_2); no longer J1.1 (Pin_1)
- net at C12.2, U2.4 (OB): now also J1.1 (Pin_1); no longer J1.2 (Pin_2)
Changed lines of the file:
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@@
 	(wire
 		(pts
-			(xy 262.89 39.37) (xy 243.84 39.37)
-		)
-		(stroke
-			(width 0)
-			(type default)
-		)
-	)
-	(wire
-		(pts
 			(xy 76.2 125.73) (xy 76.2 129.54)
 		)
@@
 	(wire
 		(pts
-			(xy 247.65 41.91) (xy 262.89 41.91)
-		)
-		(stroke
-			(width 0)
-			(type default)
-		)
-	)
-	(wire
-		(pts
-			(xy 243.84 41.91) (xy 241.3 41.91)
+			(xy 241.3 41.91) (xy 262.89 41.91)
 		)
 		(stroke
@@
 	(wire
 		(pts
+			(xy 247.65 34.29) (xy 247.65 39.37)
+		)
+		(stroke
+			(width 0)
+			(type default)
+		)
+	)
+	(wire
+		(pts
 			(xy 138.43 152.4) (xy 140.97 152.4)
 		)
@@
 	(wire
 		(pts
+			(xy 247.65 39.37) (xy 262.89 39.37)
+		)
+		(stroke
+			(width 0)
+			(type default)
+		)
+	)
+	(wire
+		(pts
 			(xy 59.69 26.67) (xy 59.69 31.75)
 		)
@@
 	(wire
 		(pts
-			(xy 247.65 34.29) (xy 247.65 41.91)
-		)
-		(stroke
-			(width 0)
-			(type default)
-		)
-	)
-	(wire
-		(pts
 			(xy 69.85 115.57) (xy 77.47 115.57)
 		)
@@
 	(wire
 		(pts
-			(xy 243.84 39.37) (xy 243.84 41.91)
-		)
-		(stroke
-			(width 0)
-			(type default)
-		)
-	)
-	(wire
-		(pts
 			(xy 20.32 66.04) (xy 21.59 66.04)
 		)
@@
 			)
 		)
-		(property "Footprint" "TestPoint:TestPoint_Pad_1.0x1.0mm"
+		(property "Footprint" "TestPoint:TestPoint_Pad_D1.0mm"
 			(at 110.49 22.86 0)
 			(effects

Commit message: rf begins...
Connections:
- net at U1.11 (GPIO10): now also U2.6 (IA); no longer U2.7 (IB)
- net at U1.12 (GPIO11): now also U2.7 (IB); no longer U2.6 (IA)
Changed lines of the file:
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@@
-	(wire
-		(pts
-			(xy 215.9 41.91) (xy 207.01 41.91)
-		)
-		(stroke
-			(width 0)
-			(type default)
-		)
-	)
 	(wire
 		(pts
@@
 	(wire
 		(pts
-			(xy 215.9 38.1) (xy 215.9 34.29)
-		)
-		(stroke
-			(width 0)
-			(type default)
-		)
-	)
-	(wire
-		(pts
 			(xy 161.29 64.77) (xy 165.1 64.77)
 		)
@@
 	(wire
 		(pts
-			(xy 207.01 34.29) (xy 199.39 34.29)
+			(xy 199.39 34.29) (xy 215.9 34.29)
 		)
 		(stroke
@@
 	(wire
 		(pts
-			(xy 201.93 38.1) (xy 215.9 38.1)
-		)
-		(stroke
-			(width 0)
-			(type default)
-		)
-	)
-	(wire
-		(pts
-			(xy 207.01 41.91) (xy 207.01 34.29)
+			(xy 201.93 41.91) (xy 215.9 41.91)
 		)
 		(stroke
@@
 	(wire
 		(pts
-			(xy 201.93 38.1) (xy 201.93 54.61)
-		)
-		(stroke
+			(xy 201.93 41.91) (xy 201.93 54.61)
+		)
+		(stroke
