File: LockUp/_autosave-LockUp.kicad_sch (KiCad schematic)
At the start: 41 parts, among them J2 Motor, J4 Key_Sw, J5 DND_sw, J7 Servo, Q1 AO3401A, Q3 AO3400A, U1 ESP32-C6-WROOM-1, U2 L9110S, U3 MFRC522{slash}RC522, U4 L9110S

Commit message: almost...
Parts:
- added R7, R8: 47K, symbol Device:R
- R1, R2: value R -> 1K
Connections:
- net +BATT: now also R7.1
- net GND: now also R8.2
- net at U1.27 (GPIO2/ADC1_CH2): now also R7.2, R8.1
Other:
- company: (none) -> Ornex
- title: (none) -> Ornex Z-Lock
- moved on the sheet: 300R1, 300R2, 5K1, 820R1, J5, J7, NC16, NC17, NC18, NC19, NC20, NC21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
