File: LockUp/_autosave-conn.kicad_sch (KiCad schematic)
At the start: 12 parts, among them J3 Usb_Pwr, J6 Bat_Pwr, Q2 Si2323, U15 TPS63802DLAR

Commit message: almost...
Other:
- company: (none) -> Ornex
Changed lines of the file:
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@@
 	(generator_version "9.0")
 	(paper "A4")
+	(title_block
+		(date "2025-06-05")
+		(rev "0.0.1")
+		(company "Ornex")
+	)
 	(text_box "Защита от переполюсовки, защита батареи от обратки ЮСБ"
 		(exclude_from_sim no)
