File: LockUp/conn.kicad_sch (KiCad schematic)
At the start: 12 parts, among them J3 Usb_Pwr, J6 Bat_Pwr, Q2 Si2323, U15 TPS63802DLAR

Commit message: bat mon done
Parts:
- C1, C2: footprint Capacitor_SMD:C_0603_1608Metric -> Capacitor_SMD:C_0805_2012Metric_Pad1.18x1.45mm_HandSolder
- R3, R4, R5, R6: footprint Resistor_SMD:R_0603_1608Metric -> Resistor_SMD:R_0805_2012Metric_Pad1.20x1.40mm_HandSolder
Other:
- company: (none) -> Ornex
- title: (none) -> Ornex Z-Lock
- moved on the sheet: C2, R4
Changed lines of the file:
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@@
 	(generator_version "9.0")
 	(paper "A4")
+	(title_block
+		(title "Ornex Z-Lock")
+		(date "2025-06-05")
+		(rev "0.0.3")
+		(company "Ornex")
+		(comment 1 "Схема питания")
+	)
 	(text_box "Защита от переполюсовки, защита батареи от обратки ЮСБ"
 		(exclude_from_sim no)
@@
 	(wire
 		(pts
-			(xy 152.4 52.07) (xy 152.4 63.5)
+			(xy 152.4 55.88) (xy 152.4 63.5)
 		)
 		(stroke
@@
 	(wire
 		(pts
-			(xy 144.78 50.8) (xy 144.78 55.88)
+			(xy 144.78 53.34) (xy 144.78 55.88)
 		)
 		(stroke
@@
 	(wire
 		(pts
-			(xy 152.4 43.18) (xy 152.4 46.99)
+			(xy 152.4 43.18) (xy 152.4 50.8)
 		)
 		(stroke
@@
 		(pts
 			(xy 64.77 43.18) (xy 69.85 43.18)
+		)
+		(stroke
+			(width 0)
+			(type default)
+		)
+	)
+	(wire
+		(pts
+			(xy 144.78 45.72) (xy 144.78 43.18)
 		)
 		(stroke
@@
 					(size 1.27 1.27)
 				)
+				(hide yes)
 			)
 		)
@@
 			)
 		)
-		(property "Footprint" "Resistor_SMD:R_0603_1608Metric"
+		(property "Footprint" "Resistor_SMD:R_0805_2012Metric_Pad1.20x1.40mm_HandSolder"
 			(at 57.912 57.15 90)
 			(effects
@@
 				)
 				(justify right)
+				(hide yes)
 			)
 		)
@@
 					(size 1.27 1.27)
 				)
+				(hide yes)
 			)
 		)
@@
 			)
 		)
-		(property "Footprint" "Resistor_SMD:R_0603_1608Metric"
+		(property "Footprint" "Resistor_SMD:R_0805_2012Metric_Pad1.20x1.40mm_HandSolder"
 			(at 135.382 46.99 90)
 			(effects
@@
 				)
 				(justify right)
+				(hide yes)
 			)
 		)
@@
 		(on_board yes)
 		(dnp no)
-		(fields_autoplaced yes)
 		(property "Reference" "Q2"
-			(at 59.69 36.83 90)
+			(at 59.944 39.116 90)
 			(effects
 				(font
@@
 					(size 1.27 1.27)
 				)
+				(hide yes)
 			)
 		)
@@
 	(symbol
 		(lib_id "Device:R")
-		(at 144.78 46.99 0)
+		(at 144.78 49.53 0)
 		(unit 1)
 		(exclude_from_sim no)
@@
 		(dnp no)
 		(property "Reference" "R4"
-			(at 148.59 45.72 0)
+			(at 148.59 48.26 0)
 			(effects
 				(font
@@
 		)
 		(property "Value" "560k"
-			(at 148.59 48.26 0)
-			(effects
-				(font
-					(size 1.27 1.27)
-				)
-			)
-		)
-		(property "Footprint" "Resistor_SMD:R_0603_1608Metric"
-			(at 143.002 46.99 90)
+			(at 148.59 50.8 0)
+			(effects
+				(font
+					(size 1.27 1.27)
+				)
+			)
+		)
+		(property "Footprint" "Resistor_SMD:R_0805_2012Metric_Pad1.20x1.40mm_HandSolder"
+			(at 143.002 49.53 90)
 			(effects
 				(font
@@
 		)
 		(property "Datasheet" "~"
-			(at 144.78 46.99 0)
+			(at 144.78 49.53 0)
 			(effects
 				(font
@@
 		)
 		(property "Description" ""
-			(at 144.78 46.99 0)
+			(at 144.78 49.53 0)
 			(effects
 				(font
@@
 		)
 		(property "LCSC Part #" "C101109"
-			(at 144.78 46.99 0)
+			(at 144.78 49.53 0)
 			(effects
 				(font
@@
 					(size 1.27 1.27)
 				)
+				(hide yes)
 			)
 		)
@@
 					(size 1.27 1.27)
 				)
+				(hide yes)
 			)
 		)
@@
 	(symbol
 		(lib_id "Device:C_Small")
-		(at 152.4 49.53 0)
+		(at 152.4 53.34 0)
 		(unit 1)
 		(exclude_from_sim no)
@@
 		(dnp no)
 		(property "Reference" "C2"
-			(at 154.94 48.26 0)
+			(at 154.94 52.07 0)
 			(effects
 				(font
@@
 		)
 		(property "Value" "22uF"
-			(at 154.94 50.8 0)
+			(at 154.94 54.61 0)
 			(effects
 				(font
@@
 			)
 		)
-		(property "Footprint" "Capacitor_SMD:C_0603_1608Metric"
-			(at 152.4 49.53 0)
+		(property "Footprint" "Capacitor_SMD:C_0805_2012Metric_Pad1.18x1.45mm_HandSolder"
+			(at 152.4 53.34 0)
 			(effects
 				(font
@@
 		)
 		(property "Datasheet" "~"
-			(at 152.4 49.53 0)
+			(at 152.4 53.34 0)
 			(effects
 				(font
@@
 		)
 		(property "Description" ""
-			(at 152.4 49.53 0)
+			(at 152.4 53.34 0)
 			(effects
 				(font
@@
 		)
 		(property "LCSC Part #" "C59461"
-			(at 152.4 49.53 0)
+			(at 152.4 53.34 0)
 			(effects
 				(font
@@
 			)
 		)
-		(property "Footprint" "Capacitor_SMD:C_0603_1608Metric"
+		(property "Footprint" "Capacitor_SMD:C_0805_2012Metric_Pad1.18x1.45mm_HandSolder"
 			(at 87.63 48.26 0)
 			(effects
@@
 			)
 		)
-		(property "Footprint" "Resistor_SMD:R_0603_1608Metric"
+		(property "Footprint" "Resistor_SMD:R_0805_2012Metric_Pad1.20x1.40mm_HandSolder"
 			(at 143.002 59.69 90)
 			(effects

Commit message: fucked up
Parts:
- added D2: 1N4001W, Diode_SMD:D_SOD-123F, symbol Device:D_Small
Connections:
- net +BATT: now also D2.2 (A)
- net at C1.1, D1.1 (K), Q2.2 (S)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: now also D2.1 (K)
Changed lines of the file:
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@@
 		(title "Ornex Z-Lock")
 		(date "2025-06-05")
-		(rev "0.0.3")
+		(rev "0.0.4")
 		(company "Ornex")
 		(comment 1 "Схема питания")
@@
 	)
 	(junction
+		(at 50.8 43.18)
+		(diameter 0)
+		(color 0 0 0 0)
+	)
+	(junction
 		(at 69.85 52.07)
 		(diameter 0)
@@
 	(wire
 		(pts
-			(xy 35.56 43.18) (xy 54.61 43.18)
+			(xy 35.56 43.18) (xy 50.8 43.18)
 		)
 		(stroke
@@
 	(wire
 		(pts
+			(xy 69.85 33.02) (xy 69.85 43.18)
+		)
+		(stroke
+			(width 0)
+			(type default)
+		)
+	)
+	(wire
+		(pts
 			(xy 132.08 63.5) (xy 144.78 63.5)
 		)
@@
 	(wire
 		(pts
+			(xy 62.23 33.02) (xy 69.85 33.02)
+		)
+		(stroke
+			(width 0)
+			(type default)
+		)
+	)
+	(wire
+		(pts
 			(xy 33.02 45.72) (xy 29.21 45.72)
 		)
@@
 	(wire
 		(pts
+			(xy 50.8 33.02) (xy 50.8 43.18)
+		)
+		(stroke
+			(width 0)
+			(type default)
+		)
+	)
+	(wire
+		(pts
 			(xy 97.79 48.26) (xy 97.79 43.18)
 		)
@@
 	(wire
 		(pts
+			(xy 57.15 33.02) (xy 50.8 33.02)
+		)
+		(stroke
+			(width 0)
+			(type default)
+		)
+	)
+	(wire
+		(pts
 			(xy 27.94 81.28) (xy 69.85 81.28)
 		)
@@
 		(pts
 			(xy 64.77 43.18) (xy 69.85 43.18)
+		)
+		(stroke
+			(width 0)
+			(type default)
+		)
+	)
+	(wire
+		(pts
+			(xy 50.8 43.18) (xy 54.61 43.18)
 		)
 		(stroke
@@
 					(unit 1)
 				)
+			)
+		)
+	)
+	(symbol
+		(lib_id "Device:D_Small")
+		(at 59.69 33.02 180)
+		(unit 1)
+		(exclude_from_sim no)
+		(in_bom yes)
+		(on_board yes)
+		(dnp no)
+		(fields_autoplaced yes)
+		(property "Reference" "D2"
+			(at 59.69 26.67 0)
+			(effects
+				(font
+					(size 1.27 1.27)
+				)
+			)
+		)
+		(property "Value" "1N4001W"
+			(at 59.69 29.21 0)
+			(effects
+				(font
+					(size 1.27 1.27)
+				)
+			)
+		)
+		(property "Footprint" "Diode_SMD:D_SOD-123F"
+			(at 59.69 33.02 90)
+			(effects
+				(font
+					(size 1.27 1.27)
+				)
+				(hide yes)
+			)
+		)
+		(property "Datasheet" "~"
+			(at 59.69 33.02 90)
+			(effects
+				(font
+					(size 1.27 1.27)
+				)
+				(hide yes)
+			)
+		)
+		(property "Description" "Diode, small symbol"
+			(at 59.69 33.02 0)
+			(effects
+				(font
+					(size 1.27 1.27)
+				)
+				(hide yes)
+			)
+		)
+		(property "Sim.Device" "D"
+			(at 59.69 33.02 0)
+			(effects
+				(font
+					(size 1.27 1.27)
+				)
+				(hide yes)
+			)
+		)
+		(property "Sim.Pins" "1=K 2=A"
+			(at 59.69 33.02 0)
+			(effects
+				(font
+					(size 1.27 1.27)
+				)
+				(hide yes)
+			)
+		)
+		(pin "2"
+		)
+		(pin "1"
+		)
+		(instances
+			(project ""
+				(path "/9f2025fc-5444-4159-a022-f8fe4f560289/e8665c0a-7ab7-4f21-9417-5f355a5b6685"
+					(reference "D2")
+					(unit 1)
+				)
