File: LockUp/LockUp.kicad_pcb (KiCad board)
At the start: 2 copper layers, 41.9 x 68.6 mm, 35 parts, among them J1 Conn_01x05_Socket, J2 Conn_01x02_Socket, U1 ESP32-C6-WROOM-1, U1 MFRC522/RC522

Commit message: bat mon done
Parts:
- moved 300R2 6.85 mm to (145.7, 94.8)
- moved NC25 6.85 mm to (137.8, 99.1)
- moved NT5 6.85 mm to (128.6, 90.8)
- moved NT6 6.85 mm to (130.3, 90.8)
- moved NC16 6.85 mm to (132.1, 103.9)
- moved NC18 6.85 mm to (139.8, 95.0)
- moved NC21 6.85 mm to (141.7, 99.1)
- moved NC22 6.85 mm to (143.8, 95.2)
- moved NC26 6.85 mm to (132.7, 94.4)
- moved NT1 6.85 mm to (123.7, 90.8)
- moved NT2 6.85 mm to (125.4, 90.8)
- moved NT4 6.85 mm to (122.1, 90.8)
- moved NY1 6.85 mm to (128.1, 103.5)
- moved 10K1 6.85 mm to (128.5, 93.7)
- moved 300R1 6.85 mm to (145.4, 99.1)
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Routing:
- net (no net): track 19.3 -> 0.03 mm, vias 2 -> 0
- net Net-(U1-GPIO8): track 0.00 -> 11.2 mm
- net Net-(NC18-Pad2): track 0.00 -> 7.98 mm, vias 0 -> 2

Commit message: fucked up
Parts:
- removed 10K1: NR14, Resistor_SMD:R_0805_2012Metric_Pad1.20x1.40mm_HandSolder
- removed 300R1: NR18, Resistor_SMD:R_0805_2012Metric_Pad1.20x1.40mm_HandSolder
- removed 300R2: NR17, Resistor_SMD:R_0805_2012Metric_Pad1.20x1.40mm_HandSolder
- removed 5K1: NR16, Resistor_SMD:R_0805_2012Metric_Pad1.20x1.40mm_HandSolder
- removed 820R1: NR15, Resistor_SMD:R_0805_2012Metric_Pad1.20x1.40mm_HandSolder
- removed J1: Conn_01x05_Socket, Connector_Molex:Molex_PicoBlade_53398-0571_1x05-1MP_P1.25mm_Vertical
- removed REF** (x2): MountingHole_3.2mm_M3_DIN965_Pad_TopOnly, MountingHole:MountingHole_3.2mm_M3_DIN965_Pad_TopOnly
- removed the U1 at (128.4, 98.0)
- added C1: 10uF, Capacitor_SMD:C_0805_2012Metric_Pad1.18x1.45mm_HandSolder, F.Cu at (210.4, 74.9)
- added C2: 22uF, Capacitor_SMD:C_0805_2012Metric_Pad1.18x1.45mm_HandSolder, F.Cu at (210.4, 77.9)
- added C3: 180pF, Capacitor_SMD:C_0805_2012Metric_Pad1.18x1.45mm_HandSolder, F.Cu at (158.1, 74.9)
- added C4: 10nF, Capacitor_SMD:C_0805_2012Metric_Pad1.18x1.45mm_HandSolder, F.Cu at (158.1, 77.9)
- added D1: BZV55 -C7V5, Diode_SMD:D_MiniMELF_Handsoldering, F.Cu at (198.0, 89.0)
- added D2: 1N4001W, Diode_SMD:D_SOD-123F, F.Cu at (208.2, 108.0)
- added J3: Usb_Pwr, Connector_Molex:Molex_PicoBlade_53398-0271_1x02-1MP_P1.25mm_Vertical, F.Cu at (198.0, 76.4)
- added J4: Key_Sw, Connector_Molex:Molex_PicoBlade_53398-0271_1x02-1MP_P1.25mm_Vertical, F.Cu at (160.9, 94.4)
- added J5: DND_sw, Connector_Molex:Molex_PicoBlade_53398-0271_1x02-1MP_P1.25mm_Vertical, F.Cu at (160.9, 101.4)
- added J6: Bat_Pwr, Connector_Molex:Molex_PicoBlade_53398-0271_1x02-1MP_P1.25mm_Vertical, F.Cu at (198.0, 83.3)
- added J7: Servo, Connector_Molex:Molex_PicoBlade_53398-0371_1x03-1MP_P1.25mm_Vertical, F.Cu at (180.9, 101.7)
- added JP3: PWR_CH, Jumper:SolderJumper-3_P1.3mm_Bridged12_RoundedPad1.0x1.5mm, F.Cu at (107.9, 73.7)
- added LS1: PKLCS1212E4001, Buzzer_Beeper:Buzzer_Mallory_AST1240MLQ, F.Cu at (191.8, 125.7)
- added NC2: 180pF, Capacitor_SMD:C_0805_2012Metric_Pad1.18x1.45mm_HandSolder, F.Cu at (158.1, 81.0)
- added Q1: Si2323, Package_TO_SOT_SMD:SOT-23, F.Cu at (172.5, 89.4)
- added Q2: Si2323, Package_TO_SOT_SMD:SOT-23, F.Cu at (205.7, 87.6)
- added Q3: AO3400A, Package_TO_SOT_SMD:SOT-23, F.Cu at (172.5, 94.0)
- added Q4: Si2323, Package_TO_SOT_SMD:SOT-23, F.Cu at (172.5, 98.6)
- added Q5: Si2323, Package_TO_SOT_SMD:SOT-23, F.Cu at (172.5, 103.3)
- added Q6: AO3400A, Package_TO_SOT_SMD:SOT-23, F.Cu at (172.5, 107.9)
- added R1: 1K, Resistor_SMD:R_0805_2012Metric_Pad1.20x1.40mm_HandSolder, F.Cu at (177.4, 94.4)
- added R10: 820R1, Resistor_SMD:R_0805_2012Metric_Pad1.20x1.40mm_HandSolder, F.Cu at (182.1, 97.3)
- added R11: 5K1, Resistor_SMD:R_0805_2012Metric_Pad1.20x1.40mm_HandSolder, F.Cu at (186.9, 88.5)
- added R12: 300, Resistor_SMD:R_0805_2012Metric_Pad1.20x1.40mm_HandSolder, F.Cu at (186.9, 91.4)
- added R13: 300, Resistor_SMD:R_0805_2012Metric_Pad1.20x1.40mm_HandSolder, F.Cu at (186.9, 94.4)
- added R14: 1K, Resistor_SMD:R_0805_2012Metric_Pad1.20x1.40mm_HandSolder, F.Cu at (186.9, 97.3)
- added R2: 1K, Resistor_SMD:R_0805_2012Metric_Pad1.20x1.40mm_HandSolder, F.Cu at (177.4, 97.3)
- added R3: 100k, Resistor_SMD:R_0805_2012Metric_Pad1.20x1.40mm_HandSolder, F.Cu at (205.7, 74.9)
- added R4: 560k, Resistor_SMD:R_0805_2012Metric_Pad1.20x1.40mm_HandSolder, F.Cu at (205.7, 77.9)
- added R5: 100k, Resistor_SMD:R_0805_2012Metric_Pad1.20x1.40mm_HandSolder, F.Cu at (205.7, 80.8)
- added R6: 1k, Resistor_SMD:R_0805_2012Metric_Pad1.20x1.40mm_HandSolder, F.Cu at (205.7, 83.8)
- added R7: 10K, Resistor_SMD:R_0805_2012Metric_Pad1.20x1.40mm_HandSolder, F.Cu at (182.1, 88.5)
- added R8: 10K, Resistor_SMD:R_0805_2012Metric_Pad1.20x1.40mm_HandSolder, F.Cu at (182.1, 91.4)
- added T1: GND, TestPoint:TestPoint_Pad_1.0x1.0mm, F.Cu at (201.9, 107.8)
- added T2: TX, TestPoint:TestPoint_Pad_1.0x1.0mm, F.Cu at (201.9, 110.8)
- added T3: RX, TestPoint:TestPoint_Pad_1.0x1.0mm, F.Cu at (201.9, 113.9)
- added T5: D-, TestPoint:TestPoint_Pad_1.0x1.0mm, F.Cu at (201.9, 117.0)
- added U4: L9110S, Package_SO:SOP-8_3.9x4.9mm_P1.27mm, F.Cu at (159.9, 108.8)
- J2: value Conn_01x02_Socket -> Motor
- NC16, NC17, NC18, NC19, NC20, NC21, NC22, NC23, NC24, NC25, NC26, NC27, NC5, NC6, NL4, NL5, NT1, NT2, NT3, NT4, NT5, NT6, NY1: moved to F.Cu
- U2: value ~ -> L9110S
- moved NT4 60.7 mm to (179.6, 110.3), turned to 0 degrees
- moved NY1 59.6 mm to (187.5, 108.6), turned to 0 degrees
- moved NT5 56.4 mm to (182.6, 107.3)
- moved NT6 55.9 mm to (182.6, 110.3)
- moved NT1 55.3 mm to (176.5, 107.3)
- moved NT3 55.1 mm to (179.6, 107.3)
- moved NT2 54.8 mm to (176.5, 110.3)
- moved NC17 47.3 mm to (162.9, 74.9), turned to 0 degrees
- moved NL4 43.2 mm to (177.4, 88.5)
- moved NL5 43.0 mm to (177.4, 91.4)
- moved NC26 36.5 mm to (167.7, 84.0), turned to 0 degrees
- moved NC27 35.4 mm to (167.7, 87.0)
- moved NC25 35.0 mm to (167.7, 81.0), turned to 0 degrees
- moved NC24 34.5 mm to (167.7, 77.9), turned to 0 degrees
- moved NC23 34.1 mm to (167.7, 74.9), turned to 0 degrees
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Connections:
- NC26 pad 1: 3V3 -> GND
- NC26 pad 2: GND -> VCC
- NC27 pad 1: 3V3 -> VCC
- NT5 pad 1: 3V3 -> VCC
- U1 pad 11: unconnected-(U1-GPIO10-Pad11) -> Net-(J4-Pin_1)
- U1 pad 12: unconnected-(U1-GPIO11-Pad12) -> Net-(J5-Pin_1)
- U1 pad 13: unconnected-(U1-GPIO12/USB_D--Pad13) -> Net-(U1-GPIO12/USB_D-)
- U1 pad 14: unconnected-(U1-GPIO13/USB_D+-Pad14) -> Net-(U1-GPIO13/USB_D+)
- U1 pad 16: unconnected-(U1-GPIO18-Pad16) -> PIEZO
- U1 pad 17: unconnected-(U1-GPIO19-Pad17) -> RFPD
- U1 pad 23: unconnected-(U1-GPIO15-Pad23) -> Net-(J7-Pin_1)
- U1 pad 24: unconnected-(U1-U0RXD/GPIO17-Pad24) -> Net-(U1-U0RXD/GPIO17)
- U1 pad 25: unconnected-(U1-U0TXD/GPIO16-Pad25) -> Net-(U1-U0TXD/GPIO16)
- U1 pad 26: unconnected-(U1-GPIO3/ADC1_CH3-Pad26) -> Net-(Q4-G)
- U1 pad 27: unconnected-(U1-GPIO2/ADC1_CH2-Pad27) -> MES
- U1 pad 4: Net-(J1-Pin_5) -> unconnected-(U1-MTMS/GPIO4/ADC1_CH4-Pad4)
- U1 pad 5: Net-(J1-Pin_4) -> MISO
- U1 pad 6: Net-(J1-Pin_3) -> CLK
- U1 pad 7: Net-(J1-Pin_2) -> MOSI
- U2 pad 2: VCC -> Net-(JP3-C)
- U2 pad 3: VCC -> Net-(JP3-C)
Routing:
- net (no net): track 0.03 -> 46.4 mm, vias 0 -> 2
- net 3V3: track 28.3 -> 0.00 mm, vias 3 -> 0
- net Net-(U3-OSCIN): track 7.92 -> 0.00 mm
- net Net-(NC6-Pad1): track 5.32 -> 0.00 mm
- net Net-(U3-OSCOUT): track 5.07 -> 0.00 mm
- net Net-(U1-GPIO8): track 11.2 -> 13.4 mm, vias 0 -> 1
- net Net-(10K1-Pad2): track 1.93 -> 0.00 mm
- net unconnected-(U1-EN/CHIP_PU-Pad3): track 0.00 -> 1.01 mm, vias 0 -> 1
- net GND: track 71.3 -> 70.3 mm, vias 10 -> 9

Commit message: ornex lock pcb
Parts:
- removed J4: Key_Sw, Connector_Molex:Molex_PicoBlade_53398-0271_1x02-1MP_P1.25mm_Vertical
- removed J5: DND_sw, Connector_Molex:Molex_PicoBlade_53398-0271_1x02-1MP_P1.25mm_Vertical
- removed J6: Bat_Pwr, Connector_Molex:Molex_PicoBlade_53398-0271_1x02-1MP_P1.25mm_Vertical
- removed NC2: 180pF, Capacitor_SMD:C_0805_2012Metric_Pad1.18x1.45mm_HandSolder
- removed R10: 820R1, Resistor_SMD:R_0805_2012Metric_Pad1.20x1.40mm_HandSolder
- removed R11: 5K1, Resistor_SMD:R_0805_2012Metric_Pad1.20x1.40mm_HandSolder
- removed R12, R13: 300, Resistor_SMD:R_0805_2012Metric_Pad1.20x1.40mm_HandSolder
- removed R3, R5: 100k, Resistor_SMD:R_0805_2012Metric_Pad1.20x1.40mm_HandSolder
- removed R4: 560k, Resistor_SMD:R_0805_2012Metric_Pad1.20x1.40mm_HandSolder
- added C10: 0.001u, Capacitor_SMD:C_0805_2012Metric_Pad1.18x1.45mm_HandSolder, F.Cu at (90.6, 96.7)
- added C11: 0.001u, Capacitor_SMD:C_0805_2012Metric_Pad1.18x1.45mm_HandSolder, F.Cu at (90.6, 99.7)
- added C12: 180pF, Capacitor_SMD:C_0805_2012Metric_Pad1.18x1.45mm_HandSolder, F.Cu at (90.6, 102.7)
- added C5: 10uF, Capacitor_SMD:C_0805_2012Metric_Pad1.18x1.45mm_HandSolder, B.Cu at (116.8, 110.9)
- added C6: 100n, Capacitor_SMD:C_0805_2012Metric_Pad1.18x1.45mm_HandSolder, B.Cu at (116.8, 106.0)
- added C7: 0.001u, Capacitor_SMD:C_0805_2012Metric_Pad1.18x1.45mm_HandSolder, F.Cu at (90.6, 87.6)
- added C8: 0.001u, Capacitor_SMD:C_0805_2012Metric_Pad1.18x1.45mm_HandSolder, F.Cu at (90.6, 90.6)
- added C9: 0.001u, Capacitor_SMD:C_0805_2012Metric_Pad1.18x1.45mm_HandSolder, F.Cu at (90.6, 93.7)
- added F1: Polyfuse, Fuse:Fuse_1206_3216Metric_Pad1.42x1.75mm_HandSolder, B.Cu at (137.5, 84.2)
- added J1: JST_B8B, Connector_JST:JST_PH_B8B-PH-SM4-TB_1x08-1MP_P2.00mm_Vertical, B.Cu at (129.5, 78.0)
- added L1: 0.47uH, Ornex:INDC2016X120N, B.Cu at (180.3, 150.1)
- added NR1: 820R1, Resistor_SMD:R_0805_2012Metric_Pad1.20x1.40mm_HandSolder, B.Cu at (28.2, 68.3)
- added NR2: 5K1, Resistor_SMD:R_0805_2012Metric_Pad1.20x1.40mm_HandSolder, B.Cu at (28.2, 65.4)
- added NR3: 300, Resistor_SMD:R_0805_2012Metric_Pad1.20x1.40mm_HandSolder, B.Cu at (28.2, 62.4)
- added NR4: 300, Resistor_SMD:R_0805_2012Metric_Pad1.20x1.40mm_HandSolder, B.Cu at (28.2, 59.5)
- added PR1: 100k, Resistor_SMD:R_0805_2012Metric_Pad1.20x1.40mm_HandSolder, B.Cu at (181.2, 147.3)
- added PR2: 560k, Resistor_SMD:R_0805_2012Metric_Pad1.20x1.40mm_HandSolder, B.Cu at (172.3, 147.3)
- added PR3: 100k, Resistor_SMD:R_0805_2012Metric_Pad1.20x1.40mm_HandSolder, B.Cu at (174.2, 149.2)
- added R15: 470, Resistor_SMD:R_0805_2012Metric_Pad1.20x1.40mm_HandSolder, F.Cu at (95.4, 102.3)
- added R16: 5K, Resistor_SMD:R_0805_2012Metric_Pad1.20x1.40mm_HandSolder, F.Cu at (100.1, 87.6)
- added R17: 10K, Resistor_SMD:R_0805_2012Metric_Pad1.20x1.40mm_HandSolder, F.Cu at (100.1, 90.5)
- added R18: 22, Resistor_SMD:R_0805_2012Metric_Pad1.20x1.40mm_HandSolder, F.Cu at (100.1, 93.5)
- added R19: 22, Resistor_SMD:R_0805_2012Metric_Pad1.20x1.40mm_HandSolder, F.Cu at (100.1, 96.5)
- added R9: 10K, Resistor_SMD:R_0805_2012Metric_Pad1.20x1.40mm_HandSolder, F.Cu at (95.4, 99.4)
- added SW1: RST, Button_Switch_SMD:SW_Push_1P1T_XKB_TS-1187A, B.Cu at (73.7, 41.8)
- added SW2: BOOT, Button_Switch_SMD:SW_Push_1P1T_XKB_TS-1187A, B.Cu at (73.7, 28.3)
- added SW3: NT_RST, Button_Switch_SMD:SW_Push_1P1T_XKB_TS-1187A, B.Cu at (73.7, 14.7)
- added T4: D+, TestPoint:TestPoint_THTPad_D1.0mm_Drill0.5mm, F.Cu at (73.7, 103.5)
- added T6: TX, TestPoint:TestPoint_THTPad_D1.0mm_Drill0.5mm, F.Cu at (72.4, 103.5)
- added T7: RES, TestPoint:TestPoint_Pad_1.0x1.0mm, F.Cu at (71.7, 108.0)
- added U15: TPS63802DLAR, Ornex:TPS63802DLAR, B.Cu at (177.3, 150.1)
- added U3: MFRC522/RC522, Package_DFN_QFN:HVQFN-32-1EP_5x5mm_P0.5mm_EP3.1x3.1mm, B.Cu at (115.6, 65.0)
- C1, C2, C3, C4, D1, D2, J3, J7, JP3, NC16, NC17, NC18, NC19, NC20, NC21, NC22, NC23, NC24, NC25, NC26, NC27, NC5, NC6, NL4, NL5, NT1, NT2, NT3, NT4, NT5, NT6, NY1, Q2, R6: moved to B.Cu
- J2: value Motor -> USB_B_Mini; footprint Connector_Molex:Molex_PicoBlade_53398-0271_1x02-1MP_P1.25mm_Vertical -> Connector_USB:USB_Mini-B_Wuerth_65100516121_Horizontal
- R1, R2: value 1K -> 10K
- T1, T5: footprint TestPoint:TestPoint_Pad_1.0x1.0mm -> TestPoint:TestPoint_THTPad_D1.0mm_Drill0.5mm
- T2, T3: footprint TestPoint:TestPoint_Pad_1.0x1.0mm -> TestPoint:TestPoint_Pad_D1.0mm
- moved T3 130.4 mm to (72.4, 97.9)
- moved R1 130.4 mm to (47.9, 78.4)
- moved R14 130.4 mm to (57.4, 81.3)
- moved R2 130.4 mm to (47.9, 81.3)
- moved Q1 130.4 mm to (43.1, 73.4)
- moved Q3 130.4 mm to (43.1, 78.0)
- moved T2 130.4 mm to (72.4, 94.9)
- moved T5 130.3 mm to (72.4, 102.2)
- moved T1 128.3 mm to (73.7, 102.2)
- moved NC16 124.5 mm to (39.4, 52.3)
- moved NC22 124.5 mm to (44.2, 52.3)
- moved NC21 122.8 mm to (44.2, 55.3)
- moved NC6 122.8 mm to (39.4, 55.3)
- moved NC27 122.8 mm to (49.1, 55.3)
- moved NC20 121.3 mm to (44.2, 58.3)
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Connections:
- net Net-(Q4-G) renamed ENGAGE
- net Net-(U1-GPIO12/USB_D-) renamed D-
- D1 pad 2: Net-(D1-A) -> USB_V+
- J2 pad 1: Net-(J2-Pin_1) -> USB_V+
- J2 pad 2: Net-(J2-Pin_2) -> Net-(J2-D-)
- J3 pad 1: GND -> USB_V+
- J3 pad 2: Net-(D1-A) -> GND
- Q2 pad 1: Net-(D1-A) -> USB_V+
- R1 pad 2: Net-(J4-Pin_1) -> KEY_SW
- R2 pad 2: Net-(J5-Pin_1) -> DND_SW
- R6 pad 1: Net-(D1-A) -> USB_V+
- U1 pad 11: Net-(J4-Pin_1) -> Net-(U1-GPIO10)
- U1 pad 12: Net-(J5-Pin_1) -> Net-(U1-GPIO11)
- U1 pad 14: Net-(U1-GPIO13/USB_D+) -> D+
- U1 pad 15: Net-(U1-GPIO9) -> BOOT
- U1 pad 16: PIEZO -> Net-(J7-Pin_1)
- U1 pad 17: RFPD -> PIEZO
- U1 pad 18: unconnected-(U1-GPIO20-Pad18) -> RFPD
- U1 pad 19: unconnected-(U1-GPIO21-Pad19) -> KEY_SW
- U1 pad 23: Net-(J7-Pin_1) -> DND_SW
- U1 pad 3: unconnected-(U1-EN/CHIP_PU-Pad3) -> Net-(U1-EN/CHIP_PU)
- U1 pad 4: unconnected-(U1-MTMS/GPIO4/ADC1_CH4-Pad4) -> Net-(U1-MTMS/GPIO4/ADC1_CH4)
- U2 pad 1: Net-(J2-Pin_1) -> Net-(J1-Pin_2)
- U2 pad 4: Net-(J2-Pin_2) -> Net-(J1-Pin_1)
- U2 pad 6: Net-(U1-GPIO8) -> Net-(U1-GPIO10)
- U2 pad 7: Net-(U1-GPIO9) -> Net-(U1-GPIO11)
Routing:
- net Net-(U4-OB): track 0.00 -> 398.7 mm, vias 0 -> 4
- net ANT_TX1: track 398.7 -> 0.00 mm, vias 4 -> 0
- net GND: track 70.3 -> 2.20 mm, vias 9 -> 0
- net (no net): track 46.4 -> 0.03 mm, vias 2 -> 0
- net Net-(U1-GPIO8): track 13.4 -> 0.00 mm, vias 1 -> 0
- net SDA: track 12.4 -> 0.00 mm
- net ENGAGE: track 0.00 -> 11.9 mm
- net CLK: track 8.83 -> 0.00 mm
- net Net-(NC18-Pad2): track 7.98 -> 0.00 mm, vias 2 -> 0
- net MOSI: track 7.95 -> 0.00 mm
- net MISO: track 7.69 -> 0.00 mm
- net Net-(Q4-S): track 0.00 -> 7.38 mm
- net +BATT: track 0.00 -> 6.86 mm
- net VMID: track 6.53 -> 0.00 mm
- net RX: track 6.41 -> 0.00 mm
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
Commit message: half done
Parts:
- C4: moved to F.Cu
- R17, R18, R19: moved to B.Cu
- T1, T4, T5: footprint TestPoint:TestPoint_THTPad_D1.0mm_Drill0.5mm -> Ornex:TestPoint_THTPad_D0.6mm_Drill0.3mm
- T6: value TX -> VCC; footprint TestPoint:TestPoint_THTPad_D1.0mm_Drill0.5mm -> Ornex:TestPoint_THTPad_D0.6mm_Drill0.3mm
- moved C4 104.6 mm to (141.6, 87.0), turned to 90 degrees
- moved Q1 103.0 mm to (144.8, 89.5), turned to 180 degrees
- moved Q3 102.6 mm to (145.4, 85.7), turned to 180 degrees
- moved R14 82.8 mm to (139.7, 90.2), turned to 90 degrees
- moved R9 45.5 mm to (140.2, 107.0)
- moved T6 45.0 mm to (113.4, 84.9), turned to 0 degrees
- moved T4 44.3 mm to (113.4, 83.9), turned to 90 degrees
- moved T5 43.6 mm to (112.4, 84.9), turned to 90 degrees
- moved T1 42.9 mm to (112.4, 83.9), turned to 90 degrees
- moved R17 36.0 mm to (134.6, 100.7), turned to 90 degrees
- moved R19 33.3 mm to (133.1, 91.7), turned to 180 degrees
- moved R18 33.2 mm to (133.1, 89.8), turned to 180 degrees
- moved C8 25.5 mm to (115.8, 94.0)
- moved C7 24.5 mm to (114.9, 90.2), turned to 90 degrees
- moved R16 17.4 mm to (117.5, 88.9), turned to -90 degrees
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Connections:
- T4 pad 1: D+ -> Net-(J2-D+)
- T5 pad 1: D- -> Net-(J2-D-)
Routing:
- net MES: track 4.72 -> 38.9 mm, vias 0 -> 2
- net Net-(U4-OB): track 398.7 -> 428.9 mm
- net Net-(J2-D-): track 0.00 -> 27.9 mm, vias 0 -> 3
- net Net-(J2-D+): track 0.00 -> 27.6 mm, vias 0 -> 3
- net PIEZO: track 0.00 -> 22.7 mm
- net Net-(Q1-G): track 0.00 -> 21.9 mm
- net ENGAGE: track 11.9 -> 27.9 mm, vias 0 -> 2
- net Net-(U4-OA): track 0.00 -> 14.8 mm
- net Net-(Q1-S): track 0.00 -> 12.6 mm
- net Net-(Q4-S): track 7.38 -> 16.7 mm
- net VCC: track 0.00 -> 6.43 mm
- net Net-(U1-EN/CHIP_PU): track 0.00 -> 5.23 mm
- net +BATT: track 6.86 -> 11.0 mm, vias 0 -> 1
- net D-: track 0.00 -> 3.80 mm, vias 0 -> 1
- net D+: track 0.00 -> 3.20 mm, vias 0 -> 1
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
Commit message: doesn't fit...
Parts:
- moved SW2 112.5 mm to (135.1, 122.6)
- moved SW1 90.6 mm to (142.9, 100.3)
- moved SW3 75.6 mm to (114.9, 78.1), turned to 90 degrees
- moved C1 58.3 mm to (160.7, 97.1)
- moved C2 58.3 mm to (160.9, 91.4)
- moved D1 58.3 mm to (161.5, 87.6)
- moved D2 58.3 mm to (161.5, 80.6)
- moved J3 58.3 mm to (156.4, 79.4)
- moved L1 58.3 mm to (163.7, 94.2)
- moved PR1 58.3 mm to (164.7, 91.4)
- moved PR2 58.3 mm to (155.8, 91.4)
- moved PR3 58.3 mm to (157.7, 93.3)
- moved Q2 58.3 mm to (162.2, 83.8)
- moved R6 58.3 mm to (158.3, 85.1)
- moved U15 58.3 mm to (160.8, 94.3)
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Routing:
- net +BATT: track 11.0 -> 31.6 mm, vias 1 -> 2
- net Net-(U1-GPIO8): track 0.00 -> 10.4 mm, vias 0 -> 1
- net Net-(J1-Pin_8): track 0.00 -> 6.21 mm
- net MES: track 38.9 -> 36.0 mm
- net VCC: track 6.43 -> 9.08 mm, vias 0 -> 1

Commit message: esp placed
Parts:
- U1: moved to B.Cu
- moved U1 94.0 mm to (219.7, 75.9), turned to 90 degrees
- moved J1 74.3 mm to (203.8, 76.2), turned to 90 degrees
- moved J3 39.9 mm to (196.2, 76.8)
- moved J7 23.6 mm to (163.2, 107.3)
Other:
- board size 41.9 x 68.6 mm -> 122.5 x 72.6 mm

Commit message: pre traces
Parts:
- C6, JP3: moved to F.Cu
- C7, C8, LS1, R16: moved to B.Cu
- moved C5 112.5 mm to (226.9, 87.6), turned to 0 degrees
- moved C6 111.6 mm to (226.9, 87.6), turned to 0 degrees
- moved C7 108.9 mm to (220.3, 62.9), turned to -90 degrees
- moved C8 106.6 mm to (217.8, 62.9), turned to -90 degrees
- moved NY1 102.2 mm to (218.4, 47.0)
- moved SW3 98.0 mm to (211.5, 61.0), turned to 180 degrees
- moved U3 98.0 mm to (212.1, 47.9)
- moved R16 97.6 mm to (212.1, 64.8), turned to 180 degrees
- moved R15 92.7 mm to (222.9, 84.5)
- moved R17 89.8 mm to (222.9, 87.6), turned to 180 degrees
- moved R9 89.3 mm to (226.7, 84.5), turned to 180 degrees
- moved C4 85.1 mm to (226.6, 91.5)
- moved Q4 85.1 mm to (211.6, 90.3)
- moved Q5 85.1 mm to (215.6, 89.9)
- moved Q6 85.1 mm to (207.8, 90.3)
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Routing:
- net Net-(U4-OB): track 428.9 -> 0.00 mm, vias 4 -> 0
- net MES: track 36.0 -> 0.00 mm, vias 2 -> 0
- net +BATT: track 31.6 -> 0.00 mm, vias 2 -> 0
- net ENGAGE: track 27.9 -> 0.00 mm, vias 2 -> 0
- net Net-(J2-D-): track 27.9 -> 0.00 mm, vias 3 -> 0
- net Net-(J2-D+): track 27.6 -> 0.00 mm, vias 3 -> 0
- net PIEZO: track 22.7 -> 0.00 mm
- net Net-(Q1-G): track 21.9 -> 0.00 mm
- net Net-(Q4-S): track 16.7 -> 0.00 mm
- net Net-(U4-OA): track 14.8 -> 0.00 mm
- net Net-(Q1-S): track 12.6 -> 0.00 mm
- net Net-(U1-GPIO8): track 10.4 -> 0.00 mm, vias 1 -> 0
- net VCC: track 9.08 -> 0.00 mm, vias 1 -> 0
- net Net-(J1-Pin_8): track 6.21 -> 0.00 mm
- net Net-(U1-EN/CHIP_PU): track 5.23 -> 0.00 mm
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Other:
- board size 122.5 x 72.6 mm -> 123.1 x 72.6 mm

Commit message: gate swaps...
Parts:
- removed J2: USB_B_Mini, Connector_USB:USB_Mini-B_Wuerth_65100516121_Horizontal
- C1, C2, D1, D2, L1, PR1, PR2, PR3, Q2, R18, R19, R6, U15: moved to F.Cu
- C12: moved to B.Cu
- moved C10 108.9 mm to (197.5, 76.2), turned to 90 degrees
- moved C12 106.5 mm to (196.4, 91.2), turned to 90 degrees
- moved D2 48.2 mm to (221.6, 88.9), turned to 90 degrees
- moved R6 47.4 mm to (217.2, 92.1), turned to -90 degrees
- moved Q2 46.0 mm to (218.4, 88.3), turned to 90 degrees
- moved PR2 45.4 mm to (210.8, 94.6), turned to 180 degrees
- moved D1 44.7 mm to (214.6, 88.9), turned to 90 degrees
- moved PR3 44.0 mm to (208.9, 92.7), turned to 180 degrees
- moved C2 43.7 mm to (210.8, 89.5), turned to -90 degrees
- moved U15 43.2 mm to (208.0, 89.7), turned to 90 degrees
- moved PR1 43.1 mm to (210.8, 85.7), turned to -90 degrees
- moved L1 43.1 mm to (208.0, 86.7), turned to 0 degrees
- moved C1 43.1 mm to (205.1, 89.7), turned to -90 degrees
- moved C4 18.6 mm to (217.8, 108.0), turned to 0 degrees
- moved R14 12.5 mm to (217.8, 105.4), turned to 180 degrees
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Connections:
- C12 pad 1: Net-(J1-Pin_2) -> Net-(J1-Pin_1)
- C12 pad 2: Net-(J1-Pin_1) -> Net-(J1-Pin_2)
- T6 pad 1: VCC -> USB_V+
- U2 pad 1: Net-(J1-Pin_2) -> Net-(J1-Pin_1)
- U2 pad 4: Net-(J1-Pin_1) -> Net-(J1-Pin_2)
- U2 pad 6: Net-(U1-GPIO10) -> Net-(U1-GPIO11)
- U2 pad 7: Net-(U1-GPIO11) -> Net-(U1-GPIO10)
Routing:
- net Net-(Q1-G): track 0.00 -> 23.7 mm
- net Net-(U4-OB): track 0.00 -> 18.1 mm, vias 0 -> 1
- net Net-(U1-GPIO10): track 0.00 -> 17.3 mm
- net Net-(J1-Pin_1): track 0.00 -> 15.6 mm
- net Net-(U1-GPIO11): track 0.00 -> 15.1 mm
- net Net-(J1-Pin_2): track 0.00 -> 14.9 mm
- net Net-(U4-OA): track 0.00 -> 9.61 mm, vias 0 -> 1
- net Net-(Q1-S): track 0.00 -> 2.83 mm
- net Net-(JP3-C): track 0.00 -> 1.27 mm
