File: LockUp/LockUp.kicad_pcb (KiCad board)
At the start: 2 copper layers, 123.1 x 72.6 mm, 84 parts, among them J1 JST_B8B, J3 Usb_Pwr, J7 Servo, Q1 Si2323, Q2 Si2323, Q3 AO3400A, Q4 Si2323, Q5 Si2323, Q6 AO3400A, SW1 RST, SW2 BOOT, SW3 NT_RST, T1 GND, T2 TX, T3 RX, T4 D+, T5 D-, T6 VCC, T7 RES, U1 ESP32-C6-WROOM-1, U15 TPS63802DLAR, U2 L9110S, U3 MFRC522/RC522, U4 L9110S

Commit message: frootloop day dream...
Parts:
- C5, R17, SW1, SW2: moved to F.Cu
- C9: moved to B.Cu
- T7: footprint TestPoint:TestPoint_Pad_1.0x1.0mm -> TestPoint:TestPoint_Pad_D1.0mm
- moved R2 178.1 mm to (225.9, 75.1), turned to -90 degrees
- moved R1 178.0 mm to (225.9, 79.2), turned to -90 degrees
- moved C3 171.5 mm to (207.7, 34.3)
- moved NC17 171.5 mm to (212.5, 34.3)
- moved NC18 171.5 mm to (212.5, 31.3)
- moved NC19 171.5 mm to (212.5, 28.3)
- moved NC20 171.5 mm to (212.5, 25.3)
- moved NC21 171.5 mm to (212.5, 22.3)
- moved NC22 171.5 mm to (212.5, 19.3)
- moved NC23 171.5 mm to (217.3, 34.3)
- moved NC24 171.5 mm to (217.3, 31.3)
- moved NC25 171.5 mm to (217.3, 28.3)
- moved NC26 171.5 mm to (217.3, 25.3)
- moved NC27 171.5 mm to (217.3, 22.3)
- moved NC5 171.5 mm to (207.7, 25.3)
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Connections:
- C12 pad 1: Net-(J1-Pin_1) -> Net-(J1-Pin_2)
- C12 pad 2: Net-(J1-Pin_2) -> Net-(J1-Pin_1)
- U2 pad 1: Net-(J1-Pin_1) -> Net-(J1-Pin_2)
- U2 pad 4: Net-(J1-Pin_2) -> Net-(J1-Pin_1)
Routing:
- net +BATT: track 0.00 -> 60.0 mm, vias 0 -> 3
- net Net-(J1-Pin_2): track 14.9 -> 46.1 mm, vias 0 -> 2
- net Net-(J1-Pin_1): track 15.6 -> 42.8 mm, vias 0 -> 2
- net ENGAGE: track 0.00 -> 21.3 mm, vias 0 -> 1
- net BOOT: track 0.00 -> 18.2 mm, vias 0 -> 1
- net Net-(U1-GPIO11): track 15.1 -> 30.9 mm, vias 0 -> 2
- net Net-(C11-Pad2): track 0.00 -> 14.2 mm
- net Net-(D1-K): track 0.00 -> 11.8 mm
- net Net-(U1-GPIO10): track 17.3 -> 27.8 mm, vias 0 -> 2
- net USB_V+: track 0.00 -> 9.93 mm, vias 0 -> 3
- net Net-(Q4-S): track 0.00 -> 9.27 mm, vias 0 -> 2
- net Net-(U1-EN/CHIP_PU): track 0.00 -> 7.71 mm, vias 0 -> 1
- net Net-(J1-Pin_8): track 0.00 -> 7.06 mm
- net Net-(JP3-C): track 1.27 -> 5.48 mm, vias 0 -> 1
- net Net-(Q5-S): track 0.00 -> 2.31 mm
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Other:
- board size 123.1 x 72.6 mm -> 42.5 x 69.4 mm

Commit message: rf begins...
Parts:
- added FID1: Fiducial, Fiducial:Fiducial_0.5mm_Mask1mm, F.Cu at (221.5, 108.2)
- added FID2: Fiducial, Fiducial:Fiducial_0.5mm_Mask1mm, F.Cu at (200.7, 49.5)
- added FID3: Fiducial, Fiducial:Fiducial_0.5mm_Mask1mm, B.Cu at (221.5, 108.2)
- added FID4: Fiducial, Fiducial:Fiducial_0.5mm_Mask1mm, B.Cu at (200.7, 49.5)
- added H1: MountingHole, MountingHole:MountingHole_3.2mm_M3_ISO14580, F.Cu at (193.5, 46.0)
- added H2: MountingHole, MountingHole:MountingHole_3.2mm_M3_ISO14580, F.Cu at (231.5, 108.5)
- C12, C7, C8, R16: moved to F.Cu
- T2, T3, T7: moved to B.Cu
- moved C3 70.5 mm to (212.3, 104.7)
- moved NC16 45.3 mm to (209.0, 59.2)
- moved NC6 44.2 mm to (227.9, 61.5), turned to 90 degrees
- moved T7 43.2 mm to (196.1, 65.6), turned to 90 degrees
- moved NC5 43.0 mm to (230.9, 61.5), turned to 90 degrees
- moved NR2 38.9 mm to (230.8, 50.6)
- moved NR4 38.9 mm to (230.8, 44.7)
- moved NR1 38.9 mm to (230.8, 53.6)
- moved NR3 38.9 mm to (230.8, 47.7)
- moved NC20 34.1 mm to (213.8, 59.3)
- moved NC21 34.1 mm to (213.8, 56.3)
- moved NC22 34.1 mm to (213.8, 53.3)
- moved NL5 31.3 mm to (224.0, 61.7)
- moved NC18 29.6 mm to (219.6, 60.0)
- moved NC17 29.6 mm to (219.6, 63.0)
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Connections:
- U2 pad 6: Net-(U1-GPIO11) -> Net-(U1-GPIO10)
- U2 pad 7: Net-(U1-GPIO10) -> Net-(U1-GPIO11)
Routing:
- net DND_SW: track 0.00 -> 34.6 mm, vias 0 -> 3
- net Net-(J7-Pin_1): track 0.00 -> 33.3 mm, vias 0 -> 2
- net GND: track 0.00 -> 33.3 mm, vias 0 -> 21
- net MES: track 0.00 -> 30.6 mm, vias 0 -> 1
- net USB_V+: track 9.93 -> 39.9 mm, vias 3 -> 4
- net KEY_SW: track 0.00 -> 28.2 mm, vias 0 -> 2
- net PIEZO: track 0.00 -> 25.8 mm, vias 0 -> 1
- net Net-(R18-Pad2): track 0.00 -> 25.3 mm
- net Net-(R19-Pad2): track 0.00 -> 20.9 mm, vias 0 -> 2
- net Net-(U1-MTMS/GPIO4/ADC1_CH4): track 0.00 -> 16.0 mm
- net VCC: track 0.54 -> 13.2 mm, vias 0 -> 7
- net D-: track 0.00 -> 12.5 mm, vias 0 -> 1
- net Net-(U4-OB): track 18.7 -> 29.2 mm
- net D+: track 0.00 -> 9.42 mm, vias 0 -> 1
- net Net-(Q1-G): track 23.4 -> 14.6 mm
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- added copper zone on In1.Cu, net GND
- added copper zone on In2.Cu, net VCC
Other:
- board size 42.5 x 69.4 mm -> 42.4 x 69.4 mm
- copper layers 2 -> 4
- board text added: "ANT"
