File: LockUp/power.kicad_sch (KiCad schematic)
At the start: 12 parts, among them J3 Usb_Pwr, Q2 Si2323, U15 TPS63802DLAR

Commit message: ornex lock pcb
Parts:
- added C5: 10uF, Capacitor_SMD:C_0805_2012Metric_Pad1.18x1.45mm_HandSolder, symbol Device:C_Small
- added C6: 100n, Capacitor_SMD:C_0805_2012Metric_Pad1.18x1.45mm_HandSolder, symbol Device:C_Small
- renumbered R3 to PR1, R4 to PR2, R5 to PR3
Connections:
- net GND: now also J3.2 (Pin_2), C5.2, C6.2; no longer J3.1 (Pin_1)
- net USB_V+: now also J3.1 (Pin_1); no longer J3.2 (Pin_2)
- net VCC: now also C5.1, C6.1
Other:
- note added: "или"
- moved on the sheet: J3

Commit message: rf begins...
Parts:
- added FID1, FID2, FID3, FID4: Fiducial, Fiducial:Fiducial_0.5mm_Mask1mm, symbol Mechanical:Fiducial
- added H1, H2: MountingHole, MountingHole:MountingHole_3.2mm_M3_ISO14580, symbol Mechanical:MountingHole
